Commit message: Add Camera to model and add new world

File: smt_model_description/urdf/smt_model.xacro (robot description, xacro)
@@ -124,5 +124,25 @@
     </collision>
   </link>
-  <joint name="Revolute 2" type="continuous">
+  <link name="cam_1">
+    <inertial>
+      <origin xyz="0.001500000000000043 3.136830235032246e-13 1.3877787807814457e-17" rpy="0 0 0"/>
+      <mass value="0.000665860562928387"/>
+      <inertia ixx="0.0" iyy="0.0" izz="0.0" ixy="0.0" iyz="-0.0" ixz="0.0"/>
+    </inertial>
+    <visual>
+      <origin xyz="-0.1005 0.0 -0.074" rpy="0 0 0"/>
+      <geometry>
+        <mesh filename="package://smt_model_description/meshes/cam_1.stl" scale="0.001 0.001 0.001"/>
+      </geometry>
+      <material name="silver"/>
+    </visual>
+    <collision>
+      <origin xyz="-0.1005 0.0 -0.074" rpy="0 0 0"/>
+      <geometry>
+        <mesh filename="package://smt_model_description/meshes/cam_1.stl" scale="0.001 0.001 0.001"/>
+      </geometry>
+    </collision>
+  </link>
+  <joint name="Revolute_2" type="continuous">
     <origin xyz="0.075 0.076 0.0535" rpy="0 0 0"/>
     <parent link="base_link"/>
@@ -130,5 +150,5 @@
     <axis xyz="0.0 1.0 0.0"/>
   </joint>
-  <joint name="Revolute 3" type="continuous">
+  <joint name="Revolute_3" type="continuous">
     <origin xyz="-0.075 0.076 0.0535" rpy="0 0 0"/>
     <parent link="base_link"/>
@@ -136,5 +156,5 @@
     <axis xyz="0.0 1.0 0.0"/>
   </joint>
-  <joint name="Revolute 4" type="continuous">
+  <joint name="Revolute_4" type="continuous">
     <origin xyz="-0.075 -0.076 0.0535" rpy="0 0 0"/>
     <parent link="base_link"/>
@@ -142,5 +162,5 @@
     <axis xyz="0.0 1.0 0.0"/>
   </joint>
-  <joint name="Revolute 5" type="continuous">
+  <joint name="Revolute_5" type="continuous">
     <origin xyz="0.075 -0.076 0.0535" rpy="0 0 0"/>
     <parent link="base_link"/>
@@ -153,3 +173,8 @@
     <child link="lidar_1"/>
   </joint>
+  <joint name="Rigid 8" type="fixed">
+    <origin xyz="0.1005 0.0 0.074" rpy="0 0 0"/>
+    <parent link="base_link"/>
+    <child link="cam_1"/>
+  </joint>
 </robot>

Commit message: Add new optical link for correct orientation

File: smt_model_description/urdf/smt_model.xacro (robot description, xacro)
@@ -178,3 +178,9 @@
     <child link="cam_1"/>
   </joint>
+  <joint name="camera_optical_joint" type="fixed">
+    <origin xyz="0 0 0" rpy="-1.5708 0 -1.5708"/>
+    <parent link="cam_1"/>
+    <child link="camera_link_optical"/>
+  </joint>
+  <link name="camera_link_optical" />
 </robot>

Commit message: add IMU to gazebo simulation

File: smt_model_description/urdf/smt_model.xacro (robot description, xacro)
@@ -144,4 +144,24 @@
     </collision>
   </link>
+  <link name="IMU_1">
+    <inertial>
+      <origin xyz="-5.228407822368264e-13 0.0 0.0010000000000000217" rpy="0 0 0"/>
+      <mass value="0.0012330751165340477"/>
+      <inertia ixx="0.0" iyy="0.0" izz="0.0" ixy="0.0" iyz="0.0" ixz="0.0"/>
+    </inertial>
+    <visual>
+      <origin xyz="-0.0 -0.0 -0.059" rpy="0 0 0"/>
+      <geometry>
+        <mesh filename="package://smt_model_description/meshes/IMU_1.stl" scale="0.001 0.001 0.001"/>
+      </geometry>
+      <material name="silver"/>
+    </visual>
+    <collision>
+      <origin xyz="-0.0 -0.0 -0.059" rpy="0 0 0"/>
+      <geometry>
+        <mesh filename="package://smt_model_description/meshes/IMU_1.stl" scale="0.001 0.001 0.001"/>
+      </geometry>
+    </collision>
+  </link>
   <joint name="Revolute_2" type="continuous">
     <origin xyz="0.075 0.076 0.0535" rpy="0 0 0"/>
@@ -173,8 +193,13 @@
     <child link="lidar_1"/>
   </joint>
+  <joint name="Rigid 7" type="fixed">
+    <origin xyz="0.1005 0.0 0.074" rpy="0 0 0"/>
+    <parent link="base_link"/>
+    <child link="cam_1"/>
+  </joint>
   <joint name="Rigid 8" type="fixed">
-    <origin xyz="0.1005 0.0 0.074" rpy="0 0 0"/>
-    <parent link="base_link"/>
-    <child link="cam_1"/>
+    <origin xyz="0.0 0.0 0.059" rpy="0 0 0"/>
+    <parent link="base_link"/>
+    <child link="IMU_1"/>
   </joint>
   <joint name="camera_optical_joint" type="fixed">

Commit message: correlate position of IMU according to real IMU

File: smt_model_description/urdf/smt_model.xacro (robot description, xacro)
@@ -151,5 +151,5 @@
     </inertial>
     <visual>
-      <origin xyz="-0.0 -0.0 -0.059" rpy="0 0 0"/>
+      <origin xyz="0.028 -0.0 -0.06" rpy="0 0 0"/>
       <geometry>
         <mesh filename="package://smt_model_description/meshes/IMU_1.stl" scale="0.001 0.001 0.001"/>
@@ -158,5 +158,5 @@
     </visual>
     <collision>
-      <origin xyz="-0.0 -0.0 -0.059" rpy="0 0 0"/>
+      <origin xyz="0.028 -0.0 -0.06" rpy="0 0 0"/>
       <geometry>
         <mesh filename="package://smt_model_description/meshes/IMU_1.stl" scale="0.001 0.001 0.001"/>

Commit message: edit position of imu rigid

File: smt_model_description/urdf/smt_model.xacro (robot description, xacro)
@@ -151,5 +151,5 @@
     </inertial>
     <visual>
-      <origin xyz="0.028 -0.0 -0.06" rpy="0 0 0"/>
+      <origin xyz="0.034 -0.0 -0.06" rpy="0 0 0"/>
       <geometry>
         <mesh filename="package://smt_model_description/meshes/IMU_1.stl" scale="0.001 0.001 0.001"/>
@@ -158,5 +158,5 @@
     </visual>
     <collision>
-      <origin xyz="0.028 -0.0 -0.06" rpy="0 0 0"/>
+      <origin xyz="0.034 -0.0 -0.06" rpy="0 0 0"/>
       <geometry>
         <mesh filename="package://smt_model_description/meshes/IMU_1.stl" scale="0.001 0.001 0.001"/>
@@ -199,5 +199,5 @@
   </joint>
   <joint name="Rigid 8" type="fixed">
-    <origin xyz="0.0 0.0 0.059" rpy="0 0 0"/>
+    <origin xyz="-0.034 0.0 0.059" rpy="0 0 0"/>
     <parent link="base_link"/>
     <child link="IMU_1"/>
